File: eagle/driver.sch (EAGLE design)
At the start: 39 parts, among them IC1 XMEGA128A1, IC10 ST95P08M, IC11 ST95P08M, IC12 ST95P08M, IC13 ST95P08M, IC14 ST95P08M, IC15 ST95P08M, IC16 74AHC1G32DBV, IC17 74AHC1G32DBV, IC18 74AHC1G08DBV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

Commit message: driver board layout progress
Parts:
- added IC20, IC21: 74AHC1G02DBV, 74xx-little-us:74AHC1G02DBV
- added SV6: (no value), con-lstb:MA03-2
- added SV7: (no value), con-lstb:MA03-1
Connections:
- net N$103 renamed OE
- net N$104 renamed LAT
- removed net N$105: IC4G$1.4A2, IC5G$1.1A3
- new net CLK: IC4G$1.4A2
- new net CLKA: IC1.PD7, IC21A.I0
- new net CLKB: IC1.PE7, IC20A.I0
- new net CS0: IC10G$1.!S, IC11G$1.!S, IC12G$1.!S, IC18A.O
- new net CS1: IC13G$1.!S, IC14G$1.!S, IC15G$1.!S, IC19A.O
- new net N$103: IC5G$1.1A3
- new net N$106: IC8G$1.1D6, IC9G$1.2D3, SV5.33
- new net N$108: IC8G$1.1D4, IC9G$1.2D5, SV5.35
- new net N$110: IC17A.I0, IC6G$1.2Q6
- new net N$111: IC8G$1.1D2, IC9G$1.2D7, SV5.37
- new net N$113: IC16A.I0, IC7G$1.1Q3
- new net N$118: IC8G$1.1D5, IC9G$1.2D4, SV5.36
- new net N$34: IC6G$1.2D3, IC7G$1.1D6, SV5.20
- new net N$46: IC16A.O, IC21A.I1
- new net N$52: IC6G$1.1D7, IC7G$1.2D2, SV5.15
- new net SCLK0: IC10G$1.C, IC11G$1.C, IC12G$1.C, IC20A.O
- new net SCLK1: IC13G$1.C, IC14G$1.C, IC15G$1.C, IC21A.O
- new net VSYNC0: IC1.PK2, IC18A.I1, IC6G$1.2Q5
- new net VSYNC1: IC1.PK1, IC19A.I0, IC7G$1.1Q4
- net GND: now also IC6G$1.2D8, IC7G$1.1D1, IC8G$1.2D8, IC9G$1.1D1, SV6.6, SV7.3
- net N$102: now also IC8G$1.1D7, IC9G$1.2D2, SV5.31; no longer IC10G$1.C, IC11G$1.C, IC12G$1.C
- net N$109: now also IC8G$1.1D3, IC9G$1.2D6, SV5.38; no longer IC13G$1.!S, IC14G$1.!S, IC15G$1.!S
- net N$112: now also IC8G$1.1D1, IC9G$1.2D8, SV5.40; no longer IC13G$1.C, IC14G$1.C, IC15G$1.C
- net N$16: now also IC1.PE5
- net N$19: now also IC1.PE6
- net N$30: now also IC6G$1.2D4, IC7G$1.1D5, SV5.21; no longer IC10G$1.Q, IC2G$1.1A2, IC6G$1.1Q2
- net N$40: now also IC6G$1.2D2, IC7G$1.1D7, SV5.19; no longer IC11G$1.Q, IC2G$1.2A2, IC6G$1.1Q6
- net N$42: now also IC17A.O, IC20A.I1; no longer IC10G$1.!S, IC11G$1.!S, IC12G$1.!S
- net N$44: now also IC6G$1.2D1, IC7G$1.1D8, SV5.18; no longer IC12G$1.Q, IC2G$1.3A2, IC6G$1.2Q2
- net N$50: now also IC6G$1.1D8, IC7G$1.2D1, SV5.16; no longer IC15G$1.D, IC3G$1.4A1, IC7G$1.2Q5
- net N$54: now also IC6G$1.1D6, IC7G$1.2D3, SV5.13; no longer IC14G$1.D, IC3G$1.3A1, IC7G$1.2Q1
- net N$58: now also IC6G$1.1D5, IC7G$1.2D4, SV5.12; no longer IC13G$1.D, IC3G$1.2A1, IC7G$1.1Q5
- net N$59: now also IC6G$1.1D4, IC7G$1.2D5, SV5.11; no longer IC6G$1.2Q8, IC7G$1.1Q1
- net N$60: now also IC6G$1.1D3, IC7G$1.2D6, SV5.10; no longer IC6G$1.2Q7, IC7G$1.1Q2
- net N$61: now also IC6G$1.1D2, IC7G$1.2D7, SV5.8; no longer IC6G$1.2Q6, IC7G$1.1Q3
- net N$62: now also IC6G$1.1D1, IC7G$1.2D8, SV5.7; no longer IC6G$1.2Q5, IC7G$1.1Q4
- net N$87: now also IC1.PDI_DATA, SV6.1; no longer IC8G$1.2Q8, IC9G$1.1Q1
- net N$88: now also IC1.!RESET!/PDI_CLK, SV6.5; no longer IC8G$1.2Q7, IC9G$1.1Q2
- net N$89: now also IC1.PE3, SV7.1; no longer IC8G$1.2Q6, IC9G$1.1Q3
- net N$90: now also IC1.PE2, SV7.2; no longer IC8G$1.2Q5, IC9G$1.1Q4
- net N$91: now also IC8G$1.2D4, IC9G$1.1D5, SV5.24; no longer IC6G$1.2D8, IC7G$1.1D1
- net N$92: now also IC8G$1.2D7, IC9G$1.1D2, SV5.5
- net N$93: now also IC8G$1.2D6, IC9G$1.1D3, SV5.28
- net N$94: now also IC8G$1.2D5, IC9G$1.1D4, SV5.3
- net N$95: now also IC8G$1.2D3, IC9G$1.1D6, SV5.23; no longer IC8G$1.2D8, IC9G$1.1D1
- net N$96: now also IC8G$1.2D2, IC9G$1.1D7, SV5.26; no longer IC8G$1.2D7, IC9G$1.1D2
- net N$97: now also IC8G$1.2D1, IC9G$1.1D8, SV5.29; no longer IC8G$1.2D6, IC9G$1.1D3
- net N$98: now also IC8G$1.1D8, IC9G$1.2D1, SV5.32; no longer IC8G$1.2D5, IC9G$1.1D4
- net N$99: now also IC16A.I1, IC17A.I1, SV5.27
- net PH6: now also IC18A.I0
- net PJ1: now also IC19A.I1
- net PJ2: now also IC13G$1.D, IC3G$1.2A1, IC7G$1.1Q5
- net PJ3: now also IC14G$1.D, IC3G$1.3A1, IC7G$1.2Q1
- net PJ4: now also IC15G$1.D, IC3G$1.4A1, IC7G$1.2Q5
- net PJ5: now also IC10G$1.Q, IC2G$1.1A2, IC6G$1.1Q2
- net PJ6: now also IC11G$1.Q, IC2G$1.2A2, IC6G$1.1Q6
- net PJ7: now also IC12G$1.Q, IC2G$1.3A2, IC6G$1.2Q2
- net VCC: now also SV6.2

Commit message: board layout progress
Parts:
- removed IC18, IC19: 74AHC1G08DBV, 74xx-little-us:74AHC1G08DBV
Connections:
- removed net CLK: IC4G$1.4A2
- removed net CS0: IC10G$1.!S, IC11G$1.!S, IC12G$1.!S, IC18A.O
- removed net CS1: IC13G$1.!S, IC14G$1.!S, IC15G$1.!S, IC19A.O
- removed net N$103: IC5G$1.1A3
- net CLKA: now also IC4G$1.4A2
- net CLKB: now also IC5G$1.1A3
- net GND: now also IC20P.GND, IC21P.GND; no longer IC18P.GND, IC19P.GND
- net LAT: now also IC1.PE0
- net N$100: now also IC1.PK3
- net N$101: now also IC1.PK4
- net N$99: now also IC1.PR1(XT1)
- net OE: now also IC1.PE1
- net PH6: no longer IC18A.I0
- net PJ1: no longer IC19A.I1
- net VCC: now also IC20P.VCC, IC21P.VCC; no longer IC18P.VCC, IC19P.VCC
- net VSYNC0: now also IC10G$1.!S, IC11G$1.!S, IC12G$1.!S; no longer IC18A.I1
- net VSYNC1: now also IC13G$1.!S, IC14G$1.!S, IC15G$1.!S; no longer IC19A.I0

Commit message: board layout progress
Parts:
- added IC18, IC19: 74AHC1G125DBV, 74xx-little-us:74AHC1G125DBV
- added IC22, IC23, IC24, IC25: ST95P08M, st-microelectronics:ST95P08M
- added R4, R5: 33k, rcl:R-US_R0402
- IC16, IC17: value 74AHC1G32DBV -> 74AHC1G02DBV; device 74xx-little-us:74AHC1G32DBV -> 74xx-little-us:74AHC1G02DBV
- IC20, IC21: value 74AHC1G02DBV -> ST95P08M; device 74xx-little-us:74AHC1G02DBV -> st-microelectronics:ST95P08M
Connections:
- removed net CLKA: IC1.PD7, IC21A.I0, IC4G$1.4A2
- removed net CLKB: IC1.PE7, IC20A.I0, IC5G$1.1A3
- removed net N$100: IC1.PK3, IC7G$1.1OE, IC7G$1.2OE, IC9G$1.1OE, IC9G$1.2OE
- removed net N$101: IC1.PK4, IC6G$1.1OE, IC6G$1.2OE, IC8G$1.1OE, IC8G$1.2OE
- removed net N$75: IC5G$1.4A4, IC9G$1.2Q8
- removed net N$77: IC5G$1.4A2, IC9G$1.2Q6
- removed net N$79: IC5G$1.3A4, IC9G$1.2Q4
- removed net N$81: IC5G$1.3A2, IC9G$1.2Q2
- removed net N$83: IC5G$1.2A4, IC9G$1.1Q8
- removed net N$85: IC5G$1.2A2, IC9G$1.1Q6
- new net CLK_EN0: IC1.PK5, IC19A.OE
- new net CLK_EN1: IC1.PK6, IC18A.OE
- new net N$48: IC1.PK3, IC6G$1.1OE, IC6G$1.2OE, IC9G$1.1OE, IC9G$1.2OE
- new net N$56: IC1.PK4, IC7G$1.1OE, IC7G$1.2OE, IC8G$1.1OE, IC8G$1.2OE
- new net PB0: IC1.PB0, IC25G$1.D, IC5G$1.2A4, IC9G$1.1Q8
- new net PB1: IC1.PB1, IC24G$1.D, IC5G$1.3A4, IC9G$1.2Q4
- new net PB2: IC1.PB2, IC23G$1.D, IC5G$1.4A4, IC9G$1.2Q8
- new net PB3: IC1.PB3, IC25G$1.Q, IC5G$1.2A2, IC9G$1.1Q6
- new net PB4: IC1.PB4, IC24G$1.Q, IC5G$1.3A2, IC9G$1.2Q2
- new net PB5: IC1.PB5, IC23G$1.Q, IC5G$1.4A2, IC9G$1.2Q6
- new net PB6: IC1.PB6
- new net PB7: IC1.PB7
- new net VSYNC2: IC1.PA6, IC20G$1.!S, IC21G$1.!S, IC22G$1.!S, IC8G$1.2Q5
- new net VSYNC3: IC1.PA7, IC23G$1.!S, IC24G$1.!S, IC25G$1.!S, IC9G$1.1Q4
- net GND: now also IC18P.GND, IC19P.GND, IC22P.GND, IC23P.GND, IC24P.GND, IC25P.GND
- net N$110: now also R4.1
- net N$113: now also R5.1
- net N$16: now also IC3G$1.1G, IC3G$1.2G, IC3G$1.3G, IC3G$1.4G; no longer IC2G$1.1G, IC2G$1.2G, IC2G$1.3G, IC2G$1.4G
- net N$19: now also IC2G$1.1G, IC2G$1.2G, IC2G$1.3G, IC2G$1.4G; no longer IC3G$1.1G, IC3G$1.2G, IC3G$1.3G, IC3G$1.4G
- net N$42: now also IC16A.O, IC18A.I; no longer IC17A.O, IC20A.I1
- net N$46: now also IC17A.O, IC19A.I; no longer IC16A.O, IC21A.I1
- net N$63: now also IC22G$1.D
- net N$64: now also IC22G$1.!W
- net N$65: now also IC22G$1.!HOLD
- net N$66: now also IC22G$1.Q
- net N$67: now also IC21G$1.D
- net N$68: now also IC21G$1.!W
- net N$69: now also IC21G$1.Q
- net N$70: now also IC21G$1.!HOLD
- net N$71: now also IC20G$1.D
- net N$72: now also IC20G$1.!W
- net N$73: now also IC20G$1.Q
- net N$74: now also IC20G$1.!HOLD
- net N$76: now also IC23G$1.!W
- net N$78: now also IC23G$1.!HOLD
- net N$80: now also IC24G$1.!W
- net N$82: now also IC24G$1.!HOLD
- net N$84: now also IC25G$1.!W
- net N$86: now also IC25G$1.!HOLD
- net SCLK0: now also IC1.PD7, IC19A.O, IC23G$1.C, IC24G$1.C, IC25G$1.C, IC5G$1.1A3; no longer IC20A.O
- net SCLK1: now also IC1.PE7, IC18A.O, IC20G$1.C, IC21G$1.C, IC22G$1.C, IC4G$1.4A2; no longer IC21A.O
- net VCC: now also IC18P.VCC, IC19P.VCC, IC22P.VCC, IC23P.VCC, IC24P.VCC, IC25P.VCC, R4.2, R5.2
Other:
- moved on the sheet: IC20P, IC21P

Commit message: board layout progress
Parts:
- added C13, C14, C15: 100n, rcl:C-USC0402
Connections:
- removed net N$63: IC22G$1.D, IC4G$1.1A1, IC8G$1.1Q1
- removed net N$66: IC22G$1.Q, IC4G$1.1A3, IC8G$1.1Q3
- removed net N$67: IC21G$1.D, IC4G$1.2A1, IC8G$1.1Q5
- removed net N$69: IC21G$1.Q, IC4G$1.2A3, IC8G$1.1Q7
- removed net N$71: IC20G$1.D, IC4G$1.3A1, IC8G$1.2Q1
- removed net N$73: IC20G$1.Q, IC4G$1.3A3, IC8G$1.2Q3
- new net PC0: IC1.PC0, IC22G$1.Q, IC4G$1.1A3, IC8G$1.1Q3
- new net PC1: IC1.PC1, IC21G$1.Q, IC4G$1.2A3, IC8G$1.1Q7
- new net PC2: IC1.PC2, IC20G$1.Q, IC4G$1.3A3, IC8G$1.2Q3
- new net PC3: IC1.PC3, IC22G$1.D, IC4G$1.1A1, IC8G$1.1Q1
- new net PC4: IC1.PC4, IC21G$1.D, IC4G$1.2A1, IC8G$1.1Q5
- new net PC5: IC1.PC5, IC20G$1.D, IC4G$1.3A1, IC8G$1.2Q1
- new net PC6: IC1.PC6
- new net PC7: IC1.PC7
- net GND: now also C13.2, C14.2, C15.2
- net VCC: now also C13.1, C14.1, C15.1

Commit message: board layout progress
Parts:
- added C16, C17, C18, C19: 100n, rcl:C-USC0402
- added R10, R6, R7, R8, R9: 47k, rcl:R-US_R0402
Connections:
- net GND: now also C16.2, C17.2, C18.2, C19.2, R10.2, R6.1, R7.1, R8.1, R9.1
- net N$11: now also R9.2
- net N$12: now also R10.1
- net N$15: now also R8.2
- net N$17: now also R7.2
- net N$27: now also R6.2
- net VCC: now also C16.1, C17.1, C18.1, C19.1

Commit message: board layout progress
Parts:
- added C20, C21, C22, C23: 100n, rcl:C-USC0402
- added R11, R12, R13, R14, R15, R16, R17, R18, R19, R20, R21, R22, R23, R24, R25, R26, R27, R28, R29, R30, R31, R32, R33, R34: 33k, rcl:R-US_R0402
Connections:
- net GND: now also C20.2, C21.2, C22.2, C23.2
- net N$29: now also R11.1
- net N$31: now also R12.2
- net N$35: now also R15.1
- net N$41: now also R13.2
- net N$43: now also R16.1
- net N$45: now also R14.2
- net N$47: now also R17.1
- net N$49: now also R18.2
- net N$51: now also R19.1
- net N$53: now also R20.2
- net N$55: now also R21.1
- net N$57: now also R22.2
- net N$64: now also R28.2
- net N$65: now also R27.1
- net N$68: now also R26.2
- net N$70: now also R25.1
- net N$72: now also R24.2
- net N$74: now also R23.1
- net N$76: now also R30.2
- net N$78: now also R29.1
- net N$80: now also R32.2
- net N$82: now also R31.1
- net N$84: now also R34.2
- net N$86: now also R33.1
- net PB7: now also R29.2, R30.1, R31.2, R32.1, R33.2, R34.1
- net PC7: now also R23.2, R24.1, R25.2, R26.1, R27.2, R28.1
- net PH6: now also R17.2, R18.1, R19.2, R20.1, R21.2, R22.1
- net PH7: now also R11.2, R12.1, R13.1, R14.1, R15.2, R16.2
- net VCC: now also C20.1, C21.1, C22.1, C23.1
Other:
- moved on the sheet: IC24, IC25

Commit message: finalizing board layout
Connections:
- net GND: now also IC8G$1.2D6, IC8G$1.2D7, IC9G$1.1D2, IC9G$1.1D3
- net N$92: no longer IC8G$1.2D7, IC9G$1.1D2
- net N$93: no longer IC8G$1.2D6, IC9G$1.1D3
Changed lines of the file:
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@@
 <part name="R33" library="rcl" library_urn="urn:adsk.eagle:library:334" deviceset="R-US_" device="R0402" package3d_urn="urn:adsk.eagle:package:23547/3" value="33k"/>
 <part name="R34" library="rcl" library_urn="urn:adsk.eagle:library:334" deviceset="R-US_" device="R0402" package3d_urn="urn:adsk.eagle:package:23547/3" value="33k"/>
+<part name="SUPPLY109" library="supply2" library_urn="urn:adsk.eagle:library:372" deviceset="GND" device=""/>
+<part name="SUPPLY110" library="supply2" library_urn="urn:adsk.eagle:library:372" deviceset="GND" device=""/>
 </parts>
 <sheets>
@@
 <attribute name="NAME" x="125.9586" y="222.25" size="1.778" layer="95" rot="R270"/>
 <attribute name="VALUE" x="121.158" y="222.25" size="1.778" layer="96" rot="R270"/>
+</instance>
+<instance part="SUPPLY109" gate="GND" x="78.74" y="228.6" smashed="yes" rot="R90">
+<attribute name="VALUE" x="81.915" y="226.695" size="1.778" layer="96" rot="R90"/>
+</instance>
+<instance part="SUPPLY110" gate="GND" x="76.2" y="233.68" smashed="yes" rot="R90">
+<attribute name="VALUE" x="79.375" y="231.775" size="1.778" layer="96" rot="R90"/>
 </instance>
 </instances>
@@
 <pinref part="C23" gate="G$1" pin="2"/>
 <pinref part="SUPPLY108" gate="GND" pin="GND"/>
+</segment>
+<segment>
+<pinref part="IC9" gate="G$1" pin="1D2"/>
+<pinref part="IC8" gate="G$1" pin="2D7"/>
+<wire x1="88.9" y1="243.84" x2="76.2" y2="243.84" width="0.1524" layer="91"/>
+<wire x1="76.2" y1="243.84" x2="76.2" y2="228.6" width="0.1524" layer="91"/>
+<wire x1="76.2" y1="228.6" x2="76.2" y2="213.36" width="0.1524" layer="91"/>
+<wire x1="76.2" y1="213.36" x2="88.9" y2="213.36" width="0.1524" layer="91"/>
+<pinref part="SUPPLY109" gate="GND" pin="GND"/>
+<junction x="76.2" y="228.6"/>
+</segment>
+<segment>
+<pinref part="IC9" gate="G$1" pin="1D3"/>
+<pinref part="IC8" gate="G$1" pin="2D6"/>
+<wire x1="88.9" y1="246.38" x2="73.66" y2="246.38" width="0.1524" layer="91"/>
+<wire x1="73.66" y1="246.38" x2="73.66" y2="233.68" width="0.1524" layer="91"/>
+<wire x1="73.66" y1="233.68" x2="73.66" y2="210.82" width="0.1524" layer="91"/>
+<wire x1="73.66" y1="210.82" x2="88.9" y2="210.82" width="0.1524" layer="91"/>
+<pinref part="SUPPLY110" gate="GND" pin="GND"/>
+<junction x="73.66" y="233.68"/>
 </segment>
 </net>
@@
 <wire x1="76.2" y1="289.56" x2="76.2" y2="368.3" width="0.1524" layer="91"/>
 <junction x="76.2" y="368.3"/>
-<pinref part="IC8" gate="G$1" pin="2D7"/>
-<wire x1="88.9" y1="243.84" x2="76.2" y2="243.84" width="0.1524" layer="91"/>
-<wire x1="76.2" y1="243.84" x2="76.2" y2="213.36" width="0.1524" layer="91"/>
-<pinref part="IC9" gate="G$1" pin="1D2"/>
-<wire x1="76.2" y1="213.36" x2="88.9" y2="213.36" width="0.1524" layer="91"/>
-<wire x1="76.2" y1="289.56" x2="76.2" y2="243.84" width="0.1524" layer="91"/>
-<junction x="76.2" y="289.56"/>
-<junction x="76.2" y="243.84"/>
 </segment>
 </net>
@@
 <wire x1="-27.94" y1="365.76" x2="73.66" y2="365.76" width="0.1524" layer="91"/>
 <junction x="73.66" y="365.76"/>
-<pinref part="IC8" gate="G$1" pin="2D6"/>
-<wire x1="88.9" y1="246.38" x2="73.66" y2="246.38" width="0.1524" layer="91"/>
-<wire x1="73.66" y1="246.38" x2="73.66" y2="210.82" width="0.1524" layer="91"/>
-<pinref part="IC9" gate="G$1" pin="1D3"/>
-<wire x1="73.66" y1="210.82" x2="88.9" y2="210.82" width="0.1524" layer="91"/>
-<wire x1="73.66" y1="365.76" x2="73.66" y2="246.38" width="0.1524" layer="91"/>
-<junction x="73.66" y="246.38"/>
-</segment>
-</net>
+</segment>
+</net>
