File: eagle/driver.brd (EAGLE design)
At the start: 101.6 x 76.2 mm, 104 parts, among them IC1 XMEGA128A1, IC10 ST95P08M, IC11 ST95P08M, IC12 ST95P08M, IC13 ST95P08M, IC14 ST95P08M, IC15 ST95P08M, IC16 74AHC1G02DBV, IC17 74AHC1G02DBV, IC18 74AHC1G125DBV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

Commit message: fix sram chip select pins
Connections:
- net VSYNC0 renamed !CS0
- net VSYNC1 renamed !CS1
Changed lines of the file:
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@@
 <wire x1="43.125" y1="48.315" x2="38.1" y2="53.34" width="0.254" layer="1"/>
 </signal>
-<signal name="VSYNC0">
+<signal name="!CS0">
 <contactref element="IC6" pad="19"/>
 <wire x1="27.1018" y1="59.055" x2="28.575" y2="59.055" width="0.254" layer="16"/>
@@
 <wire x1="36.695" y1="46.99" x2="36.83" y2="46.99" width="0.254" layer="1"/>
 </signal>
-<signal name="VSYNC1">
+<signal name="!CS1">
 <contactref element="IC7" pad="6"/>
 <wire x1="27.1018" y1="59.055" x2="28.575" y2="59.055" width="0.254" layer="1"/>
