File: eagle/driver3.brd (EAGLE design)
At the start: 73 x 57.1 mm, 25 parts, among them IC1 XMEGA16A4A, IC2 74AC16244, IC3 74AC16244, IC4 74LVC1G08DBV

Commit message: board layout tweak
Routing:
- net VCC: track 33.7 -> 12.4 mm
Changed lines of the file:
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@@
 <contactref element="C5" pad="1"/>
 <polygon width="0.254" layer="1" isolate="0.254">
-<vertex x="1.27" y="40.005"/>
-<vertex x="32.385" y="40.005"/>
-<vertex x="32.385" y="14.605"/>
-<vertex x="1.27" y="14.605"/>
+<vertex x="1.27" y="13.335"/>
+<vertex x="1.27" y="53.34"/>
+<vertex x="3.175" y="53.34"/>
+<vertex x="3.175" y="45.72"/>
+<vertex x="32.385" y="45.72"/>
+<vertex x="32.385" y="13.335"/>
 </polygon>
-<wire x1="2.54" y1="52.705" x2="1.27" y2="51.435" width="0.254" layer="16"/>
-<wire x1="1.27" y1="51.435" x2="1.27" y2="33.655" width="0.254" layer="16"/>
-<wire x1="1.27" y1="33.655" x2="2.54" y2="32.385" width="0.254" layer="16"/>
 <wire x1="31.835" y1="29.21" x2="33.64" y2="29.21" width="0.4064" layer="1"/>
 <wire x1="33.64" y1="29.21" x2="33.655" y2="29.195" width="0.4064" layer="1"/>
@@
 <polygon width="0.254" layer="1" isolate="0.254">
 <vertex x="1.27" y="55.88"/>
-<vertex x="1.27" y="40.64"/>
-<vertex x="33.02" y="40.64"/>
-<vertex x="33.02" y="13.97"/>
-<vertex x="1.27" y="13.97"/>
+<vertex x="1.27" y="53.975"/>
+<vertex x="3.81" y="53.975"/>
+<vertex x="3.81" y="46.355"/>
+<vertex x="33.02" y="46.355"/>
+<vertex x="33.02" y="12.7"/>
+<vertex x="1.27" y="12.7"/>
 <vertex x="1.27" y="1.27"/>
 <vertex x="71.755" y="1.27"/>
